File: hardware/SleepLight_v2.kicad_pcb (KiCad board)
At the start: 4 copper layers, 62.3 x 62.3 mm, 72 parts, among them J2 UJ20-C-H-C-1-SMT-TR, Q1 ERT-J1VG103FM, U1 ESP32-C3-WROOM-02-N4, U2 TLV73333PDBVR, U3 MCP73871-1AAI/ML, U4 TPS61222DCKT, U6 SN74AHCT1G125DBVR

Commit message: fix: ldo en pull-up resistor
Parts:
- added R4: 330k, Resistor_SMD:R_0603_1608Metric, F.Cu at (131.4, 99.8)
Connections:
- U2 pad 3: /BAT_OUT -> Net-(U2-EN)
Routing:
- net Net-(U2-EN): track 0.00 -> 1.77 mm
- net /BAT_OUT: track 26.5 -> 27.1 mm
Changed lines of the file:
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@@
 	(net 44 "unconnected-(J2-SBU1-PadA8)")
 	(net 45 "Net-(R11-Pad2)")
+	(net 46 "Net-(U2-EN)")
 	(footprint "WS2812B-16347:COM-16347_SPK"
 		(layer "F.Cu")
@@
 		)
 	)
+	(footprint "Resistor_SMD:R_0603_1608Metric"
+		(layer "F.Cu")
+		(at 131.4 99.8 180)
+		(descr "Resistor SMD 0603 (1608 Metric), square (rectangular) end terminal, IPC-7351 nominal, (Body size source: IPC-SM-782 page 72, https://www.pcb-3d.com/wordpress/wp-content/uploads/ipc-sm-782a_amendment_1_and_2.pdf), generated with kicad-footprint-generator")
+		(tags "resistor")
+		(property "Reference" "R4"
+			(at 0 -1.43 0)
+			(layer "F.SilkS")
+			(effects
+				(font
+					(size 1 1)
+					(thickness 0.15)
+				)
+			)
+		)
+		(property "Value" "330k"
+			(at 0 1.43 0)
+			(layer "F.Fab")
+			(effects
+				(font
+					(size 1 1)
+					(thickness 0.15)
+				)
+			)
+		)
+		(property "Datasheet" "~"
+			(at 0 0 0)
+			(layer "F.Fab")
+			(hide yes)
+			(effects
+				(font
+					(size 1.27 1.27)
+					(thickness 0.15)
+				)
+			)
+		)
+		(property "Description" "Resistor, small symbol"
+			(at 0 0 0)
+			(layer "F.Fab")
+			(hide yes)
+			(effects
+				(font
+					(size 1.27 1.27)
+					(thickness 0.15)
+				)
+			)
+		)
+		(property ki_fp_filters "R_*")
+		(sheetname "/")
+		(sheetfile "SleepLight_v2.kicad_sch")
+		(attr smd)
+		(fp_line
+			(start -0.237258 0.5225)
+			(end 0.237258 0.5225)
+			(stroke
+				(width 0.12)
+				(type solid)
+			)
+			(layer "F.SilkS")
+		)
+		(fp_line
+			(start -0.237258 -0.5225)
+			(end 0.237258 -0.5225)
+			(stroke
+				(width 0.12)
+				(type solid)
+			)
+			(layer "F.SilkS")
+		)
+		(fp_rect
+			(start -1.48 -0.73)
+			(end 1.48 0.73)
+			(stroke
+				(width 0.05)
+				(type solid)
+			)
+			(fill no)
+			(layer "F.CrtYd")
+		)
+		(fp_rect
+			(start -0.8 -0.4125)
+			(end 0.8 0.4125)
+			(stroke
+				(width 0.1)
+				(type solid)
+			)
+			(fill no)
+			(layer "F.Fab")
+		)
+		(fp_text user "${REFERENCE}"
+			(at 0 0 0)
+			(layer "F.Fab")
+			(effects
+				(font
+					(size 0.4 0.4)
+					(thickness 0.06)
+				)
+			)
+		)
+		(pad "1" smd roundrect
+			(at -0.825 0 180)
+			(size 0.8 0.95)
+			(layers "F.Cu" "F.Mask" "F.Paste")
+			(roundrect_rratio 0.25)
+			(net 46 "Net-(U2-EN)")
+			(pintype "passive")
+		)
+		(pad "2" smd roundrect
+			(at 0.825 0 180)
+			(size 0.8 0.95)
+			(layers "F.Cu" "F.Mask" "F.Paste")
+			(roundrect_rratio 0.25)
+			(net 4 "/BAT_OUT")
+			(pintype "passive")
+		)
+		(embedded_fonts no)
+		(model "${KICAD9_3DMODEL_DIR}/Resistor_SMD.3dshapes/R_0603_1608Metric.step"
+			(offset
+				(xyz 0 0 0)
+			)
+			(scale
+				(xyz 1 1 1)
+			)
+			(rotate
+				(xyz 0 0 0)
+			)
+		)
+	)
 	(footprint "Capacitor_SMD:C_0603_1608Metric"
 		(layer "F.Cu")
@@
 			(layers "F.Cu" "F.Mask" "F.Paste")
 			(roundrect_rratio 0.25)
-			(net 4 "/BAT_OUT")
+			(net 46 "Net-(U2-EN)")
 			(pinfunction "EN")
 			(pintype "input")
@@
 	)
 	(segment
-		(start 130.6 96.6)
-		(end 130.6 97.6)
-		(width 0.5)
-		(layer "F.Cu")
-		(net 4)
-	)
-	(segment
-		(start 130.6 97.6)
-		(end 131.05 98.05)
-		(width 0.5)
-		(layer "F.Cu")
-		(net 4)
-	)
-	(segment
 		(start 131.075 92.925)
 		(end 130.6 93.4)
@@
 	)
 	(segment
-		(start 131.05 96.15)
-		(end 130.6 96.6)
-		(width 0.5)
-		(layer "F.Cu")
-		(net 4)
-	)
-	(segment
-		(start 131.05 98.05)
-		(end 132.2825 98.05)
-		(width 0.5)
-		(layer "F.Cu")
-		(net 4)
-	)
-	(segment
 		(start 132.2 91.5)
 		(end 132.2 92.925)
@@
 	)
 	(segment
+		(start 130.6 95.7)
+		(end 130.6 99.725)
+		(width 0.5)
+		(layer "F.Cu")
+		(net 4)
+	)
+	(segment
 		(start 135.3 85)
 		(end 135.3 86.225)
@@
 		(net 4)
 	)
+	(segment
+		(start 130.6 99.725)
+		(end 130.675 99.8)
+		(width 0.5)
+		(layer "F.Cu")
+		(net 4)
+	)
 	(via
 		(at 135.3 85)
@@
 		(net 45)
 	)
+	(segment
+		(start 132.2825 99.7425)
+		(end 132.225 99.8)
+		(width 0.2)
+		(layer "F.Cu")
+		(net 46)
+	)
+	(segment
+		(start 132.2825 98.05)
+		(end 132.2825 99.7425)
+		(width 0.2)
+		(layer "F.Cu")
+		(net 46)
+	)
 	(zone

Commit message: fix: led bypass cap positioning
Parts:
- moved C14 7.83 mm to (162.7, 118.3), turned to -158 degrees
- moved C12 7.55 mm to (177.6, 87.8), turned to -68 degrees
- moved C18 7.51 mm to (144.0, 72.7), turned to 25 degrees
- moved C13 7.45 mm to (176.5, 105.9), turned to -112 degrees
- moved C10 7.19 mm to (165.6, 73.7), turned to -25 degrees
- moved C15 7.04 mm to (143.4, 117.1), turned to 156 degrees
- moved C17 6.62 mm to (132.0, 86.1), turned to 68 degrees
- moved C16 6.44 mm to (132.0, 104.7), turned to 112 degrees
Routing:
- net /LED_5V: track 61.1 -> 71.1 mm, vias 17 -> 9
- net GND: track 98.1 -> 90.4 mm, vias 31 -> 39
